File: future/model02/pcb/model02.kicad_pcb (KiCad board)
At the start: 2 copper layers, 80 x 54 mm, 54 parts, among them J1 RJ11-6P4C, J2 USB-C 16pin, J3 KS0835F socket, SW1 EN, SW2 BOOT, U1 ESP32-S3-WROOM-1-N8R2, U2 ES8388, U3 HT9170D, U4 SY8089AAAC, U5 USBLC6-2SC6, X1 3.579545MHz, Y1 WS2812B-2020

Commit message: Finish openphone -> phone-omenal rebrand in Docker and hardware files
Rename the Docker containers, set the compose project name to
phone-omenal (it previously defaulted to the directory name "server"),
and update the remaining OPEN PHONE CO. branding in the enclosure
models, PCB silkscreen, and docs.

Co-Authored-By: Claude <noreply@anthropic.com>
Claude-Session: https://claude.ai/code/session_01WUTRuri7Jc7HTyBfYXcJfk
Other:
- board text added: "PHONE-OMENAL MODEL 02"
- board text removed: "OPEN PHONE CO. MODEL 02"
Changed lines of the file:
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@@
     (effects (font (size 0.9 0.9) (thickness 0.135)))
   )
-  (gr_text "OPEN PHONE CO.  MODEL 02" (at 40 17.5) (layer "F.SilkS")
+  (gr_text "PHONE-OMENAL  MODEL 02" (at 40 17.5) (layer "F.SilkS")
     (effects (font (size 1.5 1.5) (thickness 0.224999)))
   )
